Commit message: added mesh files for Atlas for visualization

File: models/robots/Atlas/Atlas_description/urdf/atlas.urdf (robot description, URDF)
Before this commit: robot drc_skeleton, 31 links, 30 joints
Links:
- link l_clav: geometry collision mesh filename=urdf/meshes_unplugged/l_clav.obj; visual mesh filename=urdf/meshes_unplugged/l_clav.obj
- link l_foot: geometry collision mesh filename=urdf/meshes_unplugged/l_foot.obj; visual mesh filename=urdf/meshes_unplugged/l_foot.obj
- link l_larm: geometry collision mesh filename=urdf/meshes_unplugged/l_larm.obj; visual mesh filename=urdf/meshes_unplugged/l_larm.obj
- link l_lfarm: geometry collision mesh filename=urdf/meshes_unplugged/l_hand.obj; visual mesh filename=urdf/meshes_unplugged/l_hand.obj
- link l_lglut: geometry collision mesh filename=urdf/meshes_unplugged/l_lglut.obj; visual mesh filename=urdf/meshes_unplugged/l_lglut.obj
- link l_lleg: geometry collision mesh filename=urdf/meshes_unplugged/l_lleg.obj; visual mesh filename=urdf/meshes_unplugged/l_lleg.obj
- link l_scap: geometry collision mesh filename=urdf/meshes_unplugged/l_scap.obj; visual mesh filename=urdf/meshes_unplugged/l_scap.obj
- link l_talus: geometry collision mesh filename=urdf/meshes_unplugged/l_talus.obj; visual mesh filename=urdf/meshes_unplugged/l_talus.obj
- link l_uarm: geometry collision mesh filename=urdf/meshes_unplugged/l_uarm.obj; visual mesh filename=urdf/meshes_unplugged/l_uarm.obj
- link l_ufarm: geometry collision mesh filename=urdf/meshes_unplugged/l_farm.obj; visual mesh filename=urdf/meshes_unplugged/l_farm.obj
- link l_uglut: geometry collision mesh filename=urdf/meshes_unplugged/l_uglut.obj; visual mesh filename=urdf/meshes_unplugged/l_uglut.obj
- link l_uleg: geometry collision mesh filename=urdf/meshes_unplugged/l_uleg.obj; visual mesh filename=urdf/meshes_unplugged/l_uleg.obj
- link ltorso: geometry collision mesh filename=urdf/meshes_unplugged/ltorso.obj; visual mesh filename=urdf/meshes_unplugged/ltorso.obj
- link mtorso: geometry collision mesh filename=urdf/meshes_unplugged/mtorso.obj; visual mesh filename=urdf/meshes_unplugged/mtorso.obj
- link pelvis: geometry collision mesh filename=urdf/meshes_unplugged/pelvis.obj; visual mesh filename=urdf/meshes_unplugged/pelvis.obj
- link r_clav: geometry collision mesh filename=urdf/meshes_unplugged/r_clav.obj; visual mesh filename=urdf/meshes_unplugged/r_clav.obj
- link r_foot: geometry collision mesh filename=urdf/meshes_unplugged/r_foot.obj; visual mesh filename=urdf/meshes_unplugged/r_foot.obj
- link r_larm: geometry collision mesh filename=urdf/meshes_unplugged/r_larm.obj; visual mesh filename=urdf/meshes_unplugged/r_larm.obj
- link r_lfarm: geometry collision mesh filename=urdf/meshes_unplugged/r_hand.obj; visual mesh filename=urdf/meshes_unplugged/r_hand.obj
- link r_lglut: geometry collision mesh filename=urdf/meshes_unplugged/r_lglut.obj; visual mesh filename=urdf/meshes_unplugged/r_lglut.obj
- link r_lleg: geometry collision mesh filename=urdf/meshes_unplugged/r_lleg.obj; visual mesh filename=urdf/meshes_unplugged/r_lleg.obj
- link r_scap: geometry collision mesh filename=urdf/meshes_unplugged/r_scap.obj; visual mesh filename=urdf/meshes_unplugged/r_scap.obj
- link r_talus: geometry collision mesh filename=urdf/meshes_unplugged/r_talus.obj; visual mesh filename=urdf/meshes_unplugged/r_talus.obj
- link r_uarm: geometry collision mesh filename=urdf/meshes_unplugged/r_uarm.obj; visual mesh filename=urdf/meshes_unplugged/r_uarm.obj
- link r_ufarm: geometry collision mesh filename=urdf/meshes_unplugged/r_farm.obj; visual mesh filename=urdf/meshes_unplugged/r_farm.obj
- link r_uglut: geometry collision mesh filename=urdf/meshes_unplugged/r_uglut.obj; visual mesh filename=urdf/meshes_unplugged/r_uglut.obj
- link r_uleg: geometry collision mesh filename=urdf/meshes_unplugged/r_uleg.obj; visual mesh filename=urdf/meshes_unplugged/r_uleg.obj
- link utorso: geometry collision mesh filename=urdf/meshes_unplugged/utorso.obj; visual mesh filename=urdf/meshes_unplugged/utorso.obj
